Commit message: Adding all files

File: moveit_resources/robotic_arm_description/urdf/robotic_arm_assembly.urdf (robot description, URDF)
Before this commit: robot robotic_arm_assembly, 5 links, 4 joints
Links:
- added link world
- link base_link: mass 0.13522 -> 0.13521638090216
- link end_effector: mass 0.015759 -> 0.016378
- link link_1: mass 0.057308 -> 0.0504120841111778
- link link_2: mass 0.0052426 -> 0.0192259957524706
- link link_3: mass 0.0032899 -> 0.0145166053251896
Joints:
- added joint world_to_base_link=: type fixed, parent world, child base_link
- joint joint_1: origin xyz=0 0 0.036277 rpy=0 0 0 -> xyz=0 0 0.043143 rpy=0 0 0
- joint joint_2: origin xyz=-0.00515 0 0.028573 rpy=0 0 0 -> xyz=-0.00515 0 0.021707 rpy=0 0 0
- joint joint_3: axis 0 1 0 -> 0 -1 0; origin xyz=-0.0070261 0 0.039378 rpy=0 0 0 -> xyz=0.051117 0 0.04015 rpy=0 0 0
- joint joint_4: origin xyz=0.044 0 1.134E-05 rpy=0 0 0 -> xyz=0.053934 0 -0.03 rpy=0 0 0; type fixed -> continuous

Commit message: Add files via upload

File: moveit_resources/robotic_arm_description/urdf/robotic_arm_assembly.urdf (robot description, URDF)
Before this commit: robot robotic_arm_assembly, 6 links, 5 joints
Links:
- added link camera_link, mass 0.1; collision cylinder length=0.001 radius=0.01; visual cylinder length=0.01 radius=0.014
- added link gripper, mass 0.0008242; collision mesh filename=package://robotic_arm_description/meshes/gripper.STL; visual mesh filename=package://robotic_arm_description/meshes/gripper.STL
- link base_link: mass 0.13521638090216 -> 0.13522
- link end_effector: mass 0.016378 -> 0.015554
- link link_1: mass 0.0504120841111778 -> 0.050412
- link link_2: mass 0.0192259957524706 -> 0.019226
- link link_3: mass 0.0145166053251896 -> 0.014517
Joints:
- added joint camera_depth_joint: type fixed, parent world, child camera_link, origin xyz=0.18 0 0.2 rpy=0 1.57 3.14
- added joint joint_5: type continuous, parent end_effector, child gripper, origin xyz=0 -0.015925 -0.01717 rpy=0 0 0, axis -1 0 0
- joint joint_1: origin xyz=0 0 0.043143 rpy=0 0 0 -> xyz=0 0 0.0205 rpy=0 0 0
- joint joint_2: origin xyz=-0.00515 0 0.021707 rpy=0 0 0 -> xyz=-0.00515 0 0.04435 rpy=0 0 0
- joint joint_4: origin xyz=0.053934 0 -0.03 rpy=0 0 0 -> xyz=0.058386 0 -0.02 rpy=0 0 0
