Commit message: Added Robotic Arm Kinematics package

File: moveit_resources/robotic_arm_description/urdf/robotic_arm_description.urdf (robot description, URDF)
Before this commit: robot robotic_arm_assembly, 5 links, 4 joints
Links:
- added link gripper, mass 0.0008242; collision mesh filename=package://robotic_arm_description/meshes/gripper.STL; visual mesh filename=package://robotic_arm_description/meshes/gripper.STL
- link end_effector: mass 0.015759 -> 0.015554
- link link_1: mass 0.057308 -> 0.050412
- link link_2: mass 0.0052426 -> 0.019226
- link link_3: mass 0.0032899 -> 0.014517
Joints:
- added joint joint_5: type continuous, parent end_effector, child gripper, origin xyz=0 -0.015925 -0.01717 rpy=0 0 0, axis -1 0 0
- joint joint_1: origin xyz=0 0 0.036277 rpy=0 0 0 -> xyz=0 0 0.0205 rpy=0 0 0
- joint joint_2: origin xyz=-0.00515 0 0.028573 rpy=0 0 0 -> xyz=-0.00515 0 0.04435 rpy=0 0 0
- joint joint_3: axis 0 1 0 -> 0 -1 0; origin xyz=-0.0070261 0 0.039378 rpy=0 0 0 -> xyz=0.051117 0 0.04015 rpy=0 0 0
- joint joint_4: origin xyz=0.044 0 1.134E-05 rpy=0 0 0 -> xyz=0.058386 0 -0.02 rpy=0 0 0; type fixed -> continuous
